Commit message: ADD: fix finger param for URDF

File: end_effectors/common/franka_hand.xacro (robot description, xacro)
@@ -14,5 +14,6 @@
                        description_pkg:=franka_description
                        with_sc:=false
-                       no_prefix:=false">
+                       no_prefix:=false
+                       fix_finger:=false">
     <xacro:property name="ee_prefix" default="robot_"/>
     <xacro:unless value="${arm_id == ''}">
@@ -112,21 +113,35 @@
       <xacro:ee-inertials name="rightfinger" />
     </link>
-    <joint name="${ee_prefix}finger_joint1" type="prismatic">
-      <parent link="${ee_prefix}hand" />
-      <child link="${ee_prefix}leftfinger" />
-      <origin xyz="0 0 0.0584" rpy="0 0 0" />
-      <axis xyz="0 1 0" />
-      <limit effort="100" lower="0.0" upper="0.04" velocity="0.2" />
-      <dynamics damping="0.3" />
-    </joint>
-    <joint name="${ee_prefix}finger_joint2" type="prismatic">
-      <parent link="${ee_prefix}hand" />
-      <child link="${ee_prefix}rightfinger" />
-      <origin xyz="0 0 0.0584" rpy="0 0 ${pi}" />
-      <axis xyz="0 1 0" />
-      <limit effort="100" lower="0.0" upper="0.04" velocity="0.2" />
-      <mimic joint="${ee_prefix}finger_joint1" />
-      <dynamics damping="0.3" />
-    </joint>
+    <xacro:if value="$(arg fix_finger)">
+        <joint name="${ee_prefix}finger_joint1" type="fixed">
+          <parent link="${ee_prefix}hand" />
+          <child link="${ee_prefix}leftfinger" />
+          <origin xyz="0 0 0.0584" rpy="0 0 0" />
+        </joint>
+        <joint name="${ee_prefix}finger_joint2" type="fixed">
+          <parent link="${ee_prefix}hand" />
+          <child link="${ee_prefix}rightfinger" />
+          <origin xyz="0 0 0.0584" rpy="0 0 ${pi}" />
+        </joint>
+    </xacro:if>
+    <xacro:unless value="$(arg fix_finger)">
+        <joint name="${ee_prefix}finger_joint1" type="prismatic">
+          <parent link="${ee_prefix}hand" />
+          <child link="${ee_prefix}leftfinger" />
+          <origin xyz="0 0 0.0584" rpy="0 0 0" />
+          <axis xyz="0 1 0" />
+          <limit effort="100" lower="0.0" upper="0.04" velocity="0.2" />
+          <dynamics damping="0.3" />
+        </joint>
+        <joint name="${ee_prefix}finger_joint2" type="prismatic">
+          <parent link="${ee_prefix}hand" />
+          <child link="${ee_prefix}rightfinger" />
+          <origin xyz="0 0 0.0584" rpy="0 0 ${pi}" />
+          <axis xyz="0 1 0" />
+          <limit effort="100" lower="0.0" upper="0.04" velocity="0.2" />
+          <mimic joint="${ee_prefix}finger_joint1" />
+          <dynamics damping="0.3" />
+        </joint>
+    </xacro:unless>
   </xacro:macro>
 </robot>

File: end_effectors/franka_hand/franka_hand.urdf.xacro (robot description, xacro)
@@ -15,5 +15,6 @@
                      gazebo="$(arg gazebo)"
                      description_pkg="$(arg description_pkg)"
-                     with_sc="$(arg with_sc)">
+                     with_sc="$(arg with_sc)"
+                     fix_finger="$(arg fix_finger)">
    </xacro:franka_hand>
 </robot>

File: end_effectors/franka_hand/franka_hand_arguments.xacro (robot description, xacro)
@@ -25,3 +25,5 @@
   <!-- Name of the description package -->
   <xacro:arg name="description_pkg" default="franka_description" />
+  <!-- Use finger joint as fixed -->
+  <xacro:arg name="fix_finger" default="false" />
 </robot>

File: robots/common/franka_multi_robot.xacro (robot description, xacro)
@@ -28,5 +28,6 @@
                       gazebo_effort:=false
                       description_pkg:='franka_description'
-                      connected_to:='base'">
+                      connected_to:='base'
+                      fix_finger:=false">
     <xacro:include filename="$(find franka_description)/robots/common/utils.xacro" />
     <xacro:include filename="$(find franka_description)/robots/common/franka_arm.xacro" />
@@ -111,4 +112,5 @@
             description_pkg="${description_pkg}"
             with_sc="${with_sc}"
+            fix_finger="${fix_finger}"
           />
         </xacro:if>

File: robots/common/franka_robot.xacro (robot description, xacro)
@@ -29,5 +29,6 @@
                       arm_prefix:=''
                       description_pkg:='franka_description'
-                      connected_to:='base'">
+                      connected_to:='base'
+                      fix_finger:=false">
     <xacro:include filename="$(find franka_description)/robots/common/utils.xacro" />
     <xacro:include filename="$(find franka_description)/robots/common/franka_arm.xacro" />
@@ -72,4 +73,5 @@
         description_pkg="${description_pkg}"
         with_sc="${with_sc}"
+        fix_finger="${fix_finger}"
       />
     </xacro:if>
