Commit message: FIX: add "_" to  prefix

File: end_effectors/common/ee_with_one_link.xacro (robot description, xacro)
@@ -5,5 +5,6 @@
     <xacro:property name="ee_prefix" default="robot_"/>
     <xacro:unless value="${arm_id == ''}">
-      <xacro:property name="ee_prefix" value="${arm_prefix}${arm_id}_" />
+      <xacro:property name="arm_prefix_modified" value="${'' if arm_prefix == '' else arm_prefix + '_'}" />
+      <xacro:property name="ee_prefix" value="${arm_prefix_modified}${arm_id}_" />
     </xacro:unless>
     <xacro:unless value="${connected_to == ''}">

File: end_effectors/common/franka_hand.xacro (robot description, xacro)
@@ -18,5 +18,6 @@
     <xacro:property name="ee_prefix" default="robot_"/>
     <xacro:unless value="${arm_id == ''}">
-      <xacro:property name="ee_prefix" value="${arm_prefix}${arm_id}_" />
+      <xacro:property name="arm_prefix_modified" value="${'' if arm_prefix == '' else arm_prefix + '_'}" />
+      <xacro:property name="ee_prefix" value="${arm_prefix_modified}${arm_id}_" />
     </xacro:unless>
     <xacro:unless value="${connected_to == ''}">

File: robots/common/franka_arm.ros2_control.xacro (robot description, xacro)
@@ -51,13 +51,13 @@
         </joint>
       </xacro:macro>
-      <xacro:configure_joint joint_name="${arm_prefix}${arm_id}_joint1" initial_position="0.0"/>
-      <xacro:configure_joint joint_name="${arm_prefix}${arm_id}_joint2" initial_position="${-pi/4}"/>
-      <xacro:configure_joint joint_name="${arm_prefix}${arm_id}_joint3" initial_position="0.0"/>
-      <xacro:configure_joint joint_name="${arm_prefix}${arm_id}_joint4" initial_position="${-3*pi/4}"/>
-      <xacro:configure_joint joint_name="${arm_prefix}${arm_id}_joint5" initial_position="0.0"/>
-      <xacro:configure_joint joint_name="${arm_prefix}${arm_id}_joint6" initial_position="${pi/2}"/>
-      <xacro:configure_joint joint_name="${arm_prefix}${arm_id}_joint7" initial_position="${pi/4}"/>
+      <xacro:configure_joint joint_name="${arm_prefix_modified}${arm_id}_joint1" initial_position="0.0"/>
+      <xacro:configure_joint joint_name="${arm_prefix_modified}${arm_id}_joint2" initial_position="${-pi/4}"/>
+      <xacro:configure_joint joint_name="${arm_prefix_modified}${arm_id}_joint3" initial_position="0.0"/>
+      <xacro:configure_joint joint_name="${arm_prefix_modified}${arm_id}_joint4" initial_position="${-3*pi/4}"/>
+      <xacro:configure_joint joint_name="${arm_prefix_modified}${arm_id}_joint5" initial_position="0.0"/>
+      <xacro:configure_joint joint_name="${arm_prefix_modified}${arm_id}_joint6" initial_position="${pi/2}"/>
+      <xacro:configure_joint joint_name="${arm_prefix_modified}${arm_id}_joint7" initial_position="${pi/4}"/>
       <xacro:if value="${gazebo and hand}">
-        <xacro:configure_joint joint_name="${arm_prefix}${arm_id}_finger_joint1" initial_position="0.0" />
+        <xacro:configure_joint joint_name="${arm_prefix_modified}${arm_id}_finger_joint1" initial_position="0.0" />
       </xacro:if>
       <xacro:macro name="general_purpose_io" params="prefix command_interface index">
@@ -68,14 +68,14 @@
       </xacro:macro>
       <!-- Cartesian velocity interfaces -->
-      <xacro:general_purpose_io prefix="vx" command_interface="cartesian_velocity" index="0"/>
-      <xacro:general_purpose_io prefix="vy" command_interface="cartesian_velocity" index="1"/>
-      <xacro:general_purpose_io prefix="vz" command_interface="cartesian_velocity" index="2"/>
-      <xacro:general_purpose_io prefix="wx" command_interface="cartesian_velocity" index="3"/>
-      <xacro:general_purpose_io prefix="wy" command_interface="cartesian_velocity" index="4"/>
-      <xacro:general_purpose_io prefix="wz" command_interface="cartesian_velocity" index="5"/>
+      <xacro:general_purpose_io prefix="${arm_prefix_modified}vx" command_interface="cartesian_velocity" index="0"/>
+      <xacro:general_purpose_io prefix="${arm_prefix_modified}vy" command_interface="cartesian_velocity" index="1"/>
+      <xacro:general_purpose_io prefix="${arm_prefix_modified}vz" command_interface="cartesian_velocity" index="2"/>
+      <xacro:general_purpose_io prefix="${arm_prefix_modified}wx" command_interface="cartesian_velocity" index="3"/>
+      <xacro:general_purpose_io prefix="${arm_prefix_modified}wy" command_interface="cartesian_velocity" index="4"/>
+      <xacro:general_purpose_io prefix="${arm_prefix_modified}wz" command_interface="cartesian_velocity" index="5"/>
       <!-- Cartesian pose interfaces, in total 16 interfaces -->
       <xacro:macro name="loop" params="i">
         <xacro:unless value="${i == 16}">
-          <xacro:general_purpose_io prefix="${i}" command_interface="cartesian_pose_command" index="${i}"/>
+          <xacro:general_purpose_io prefix="${arm_prefix_modified}${i}" command_interface="cartesian_pose_command" index="${i}"/>
           <xacro:loop i="${i+1}"/>
         </xacro:unless>
@@ -83,6 +83,6 @@
       <xacro:loop i="0"/>
       <!-- Elbow command interfaces -->
-      <xacro:general_purpose_io prefix="joint_3_position" command_interface="elbow_command" index="0"/>
-      <xacro:general_purpose_io prefix="joint_4_sign" command_interface="elbow_command" index="1"/>
+      <xacro:general_purpose_io prefix="${arm_prefix_modified}joint_3_position" command_interface="elbow_command" index="0"/>
+      <xacro:general_purpose_io prefix="${arm_prefix_modified}joint_4_sign" command_interface="elbow_command" index="1"/>
     </ros2_control>
     <xacro:if value="${gazebo}">

File: robots/common/franka_arm.xacro (robot description, xacro)
@@ -10,5 +10,5 @@
   <xacro:macro name="franka_arm" params="arm_id arm_prefix:='' no_prefix:=false description_pkg:='franka_description' connected_to:='base' xyz:='0 0 0' rpy:='0 0 0' gazebo:='false' safety_distance:=0 joint_limits inertials kinematics accelerometer_config dynamics with_sc:=false" >
     <!-- Define a property that defaults to 'arm_prefix_arm_id' concatenated with an underscore if 'no_prefix' is not set -->
-    <xacro:property name="prefix" value="${'' if no_prefix else arm_prefix + arm_id + '_'}" />
+    <xacro:property name="prefix" value="${'' if no_prefix else arm_prefix + '_' + arm_id + '_'}" />
     <xacro:property name="with_accelerometers" value="${'false' if accelerometer_config == 'none' else 'true'}" />
     <xacro:if value="${gazebo}">

File: robots/common/franka_robot.xacro (robot description, xacro)
@@ -60,5 +60,5 @@
       <xacro:property name="connection" value="${special_connection if special_connection != '' else arm_id + '_link8'}" />
       <xacro:franka_hand
-        connected_to="${arm_prefix}${connection}"
+        connected_to="${arm_prefix}_${connection}"
         arm_id="${arm_id}"
         arm_prefix="${arm_prefix}"
@@ -96,4 +96,5 @@
       />
     </xacro:if>
+    <xacro:property name="arm_prefix_modified" value="${'' if arm_prefix == '' else arm_prefix + '_'}" />
     <!-- Definition of additional Gazebo tags -->
     <xacro:if value="${gazebo}">
@@ -106,39 +107,39 @@
           <origin xyz="${xyz}" rpy="${rpy}" />
           <parent link="${parent}" />
-          <child  link="${arm_prefix}${arm_id}_link0" />
+          <child  link="${arm_prefix_modified}${arm_id}_link0" />
         </joint>
       </xacro:if>
-      <xacro:gazebo-joint joint="${arm_prefix}${arm_id}_joint1" transmission="hardware_interface/PositionJointInterface" />
-      <xacro:gazebo-joint joint="${arm_prefix}${arm_id}_joint2" transmission="hardware_interface/PositionJointInterface" />
-      <xacro:gazebo-joint joint="${arm_prefix}${arm_id}_joint3" transmission="hardware_interface/PositionJointInterface" />
-      <xacro:gazebo-joint joint="${arm_prefix}${arm_id}_joint4" transmission="hardware_interface/PositionJointInterface" />
-      <xacro:gazebo-joint joint="${arm_prefix}${arm_id}_joint5" transmission="hardware_interface/PositionJointInterface" />
-      <xacro:gazebo-joint joint="${arm_prefix}${arm_id}_joint6" transmission="hardware_interface/PositionJointInterface" />
-      <xacro:gazebo-joint joint="${arm_prefix}${arm_id}_joint7" transmission="hardware_interface/PositionJointInterface" />
-      <xacro:gazebo-joint joint="${arm_prefix}${arm_id}_joint1" transmission="hardware_interface/VelocityJointInterface" />
-      <xacro:gazebo-joint joint="${arm_prefix}${arm_id}_joint2" transmission="hardware_interface/VelocityJointInterface" />
-      <xacro:gazebo-joint joint="${arm_prefix}${arm_id}_joint3" transmission="hardware_interface/VelocityJointInterface" />
-      <xacro:gazebo-joint joint="${arm_prefix}${arm_id}_joint4" transmission="hardware_interface/VelocityJointInterface" />
-      <xacro:gazebo-joint joint="${arm_prefix}${arm_id}_joint5" transmission="hardware_interface/VelocityJointInterface" />
-      <xacro:gazebo-joint joint="${arm_prefix}${arm_id}_joint6" transmission="hardware_interface/VelocityJointInterface" />
-      <xacro:gazebo-joint joint="${arm_prefix}${arm_id}_joint7" transmission="hardware_interface/VelocityJointInterface" />
-      <xacro:gazebo-joint joint="${arm_prefix}${arm_id}_joint1" transmission="hardware_interface/EffortJointInterface" />
-      <xacro:gazebo-joint joint="${arm_prefix}${arm_id}_joint2" transmission="hardware_interface/EffortJointInterface" />
-      <xacro:gazebo-joint joint="${arm_prefix}${arm_id}_joint3" transmission="hardware_interface/EffortJointInterface" />
-      <xacro:gazebo-joint joint="${arm_prefix}${arm_id}_joint4" transmission="hardware_interface/EffortJointInterface" />
-      <xacro:gazebo-joint joint="${arm_prefix}${arm_id}_joint5" transmission="hardware_interface/EffortJointInterface" />
-      <xacro:gazebo-joint joint="${arm_prefix}${arm_id}_joint6" transmission="hardware_interface/EffortJointInterface" />
-      <xacro:gazebo-joint joint="${arm_prefix}${arm_id}_joint7" transmission="hardware_interface/EffortJointInterface" />
+      <xacro:gazebo-joint joint="${arm_prefix_modified}${arm_id}_joint1" transmission="hardware_interface/PositionJointInterface" />
+      <xacro:gazebo-joint joint="${arm_prefix_modified}${arm_id}_joint2" transmission="hardware_interface/PositionJointInterface" />
+      <xacro:gazebo-joint joint="${arm_prefix_modified}${arm_id}_joint3" transmission="hardware_interface/PositionJointInterface" />
+      <xacro:gazebo-joint joint="${arm_prefix_modified}${arm_id}_joint4" transmission="hardware_interface/PositionJointInterface" />
+      <xacro:gazebo-joint joint="${arm_prefix_modified}${arm_id}_joint5" transmission="hardware_interface/PositionJointInterface" />
+      <xacro:gazebo-joint joint="${arm_prefix_modified}${arm_id}_joint6" transmission="hardware_interface/PositionJointInterface" />
+      <xacro:gazebo-joint joint="${arm_prefix_modified}${arm_id}_joint7" transmission="hardware_interface/PositionJointInterface" />
+      <xacro:gazebo-joint joint="${arm_prefix_modified}${arm_id}_joint1" transmission="hardware_interface/VelocityJointInterface" />
+      <xacro:gazebo-joint joint="${arm_prefix_modified}${arm_id}_joint2" transmission="hardware_interface/VelocityJointInterface" />
+      <xacro:gazebo-joint joint="${arm_prefix_modified}${arm_id}_joint3" transmission="hardware_interface/VelocityJointInterface" />
+      <xacro:gazebo-joint joint="${arm_prefix_modified}${arm_id}_joint4" transmission="hardware_interface/VelocityJointInterface" />
+      <xacro:gazebo-joint joint="${arm_prefix_modified}${arm_id}_joint5" transmission="hardware_interface/VelocityJointInterface" />
+      <xacro:gazebo-joint joint="${arm_prefix_modified}${arm_id}_joint6" transmission="hardware_interface/VelocityJointInterface" />
+      <xacro:gazebo-joint joint="${arm_prefix_modified}${arm_id}_joint7" transmission="hardware_interface/VelocityJointInterface" />
+      <xacro:gazebo-joint joint="${arm_prefix_modified}${arm_id}_joint1" transmission="hardware_interface/EffortJointInterface" />
+      <xacro:gazebo-joint joint="${arm_prefix_modified}${arm_id}_joint2" transmission="hardware_interface/EffortJointInterface" />
+      <xacro:gazebo-joint joint="${arm_prefix_modified}${arm_id}_joint3" transmission="hardware_interface/EffortJointInterface" />
+      <xacro:gazebo-joint joint="${arm_prefix_modified}${arm_id}_joint4" transmission="hardware_interface/EffortJointInterface" />
+      <xacro:gazebo-joint joint="${arm_prefix_modified}${arm_id}_joint5" transmission="hardware_interface/EffortJointInterface" />
+      <xacro:gazebo-joint joint="${arm_prefix_modified}${arm_id}_joint6" transmission="hardware_interface/EffortJointInterface" />
+      <xacro:gazebo-joint joint="${arm_prefix_modified}${arm_id}_joint7" transmission="hardware_interface/EffortJointInterface" />
       <xacro:transmission-franka-state arm_id="${arm_id}" />
       <xacro:transmission-franka-model arm_id="${arm_id}"
-         root="${arm_prefix}${arm_id}_joint1"
-         tip="${arm_prefix}${arm_id}_joint8"
+         root="${arm_prefix_modified}${arm_id}_joint1"
+         tip="${arm_prefix_modified}${arm_id}_joint8"
        />
       <xacro:if value="${ee_id == 'franka_hand'}">
-        <xacro:gazebo-joint joint="${arm_prefix}${arm_id}_finger_joint1" transmission="hardware_interface/EffortJointInterface" />
-        <xacro:gazebo-joint joint="${arm_prefix}${arm_id}_finger_joint2" transmission="hardware_interface/EffortJointInterface" />
+        <xacro:gazebo-joint joint="${arm_prefix_modified}${arm_id}_finger_joint1" transmission="hardware_interface/EffortJointInterface" />
+        <xacro:gazebo-joint joint="${arm_prefix_modified}${arm_id}_finger_joint2" transmission="hardware_interface/EffortJointInterface" />
         <!-- Friction specific material for Rubber/Rubber contact -->
-        <xacro:gazebo-friction link="${arm_prefix}${arm_id}_leftfinger" mu="1.13" />
-        <xacro:gazebo-friction link="${arm_prefix}${arm_id}_rightfinger" mu="1.13" />
+        <xacro:gazebo-friction link="${arm_prefix_modified}${arm_id}_leftfinger" mu="1.13" />
+        <xacro:gazebo-friction link="${arm_prefix_modified}${arm_id}_rightfinger" mu="1.13" />
       </xacro:if>
     </xacro:if>

File: robots/common/utils.xacro (robot description, xacro)
@@ -33,5 +33,5 @@
   <!-- ========================================================== -->
   <xacro:macro name="link_with_sc" params="name no_prefix:='false' rpy:='0 0 0' **self_collision_geometries gazebo:=false with_sc:=false with_accelerometers:=false">
-    <xacro:property name="prefix" value="${'' if no_prefix else arm_prefix + arm_id + '_'}" />
+    <xacro:property name="prefix" value="${'' if no_prefix else arm_prefix + '_' + arm_id + '_'}" />
     <!-- sub-link defining detailed meshes for collision with environment -->
     <link name="${prefix}${name}">
@@ -160,20 +160,20 @@
   <!-- ========================================================== -->
   <xacro:macro name="transmission-franka-state" params="arm_id:=fer">
-    <transmission name="${arm_prefix}${arm_id}_franka_state">
+    <transmission name="${arm_prefix}_${arm_id}_franka_state">
       <type>franka_hw/FrankaStateInterface</type>
-      <joint name="${arm_prefix}${arm_id}_joint1"><hardwareInterface>franka_hw/FrankaStateInterface</hardwareInterface></joint>
-      <joint name="${arm_prefix}${arm_id}_joint2"><hardwareInterface>franka_hw/FrankaStateInterface</hardwareInterface></joint>
-      <joint name="${arm_prefix}${arm_id}_joint3"><hardwareInterface>franka_hw/FrankaStateInterface</hardwareInterface></joint>
-      <joint name="${arm_prefix}${arm_id}_joint4"><hardwareInterface>franka_hw/FrankaStateInterface</hardwareInterface></joint>
-      <joint name="${arm_prefix}${arm_id}_joint5"><hardwareInterface>franka_hw/FrankaStateInterface</hardwareInterface></joint>
-      <joint name="${arm_prefix}${arm_id}_joint6"><hardwareInterface>franka_hw/FrankaStateInterface</hardwareInterface></joint>
-      <joint name="${arm_prefix}${arm_id}_joint7"><hardwareInterface>franka_hw/FrankaStateInterface</hardwareInterface></joint>
-      <actuator name="${arm_prefix}${arm_id}_motor1"><hardwareInterface>franka_hw/FrankaStateInterface</hardwareInterface></actuator>
-      <actuator name="${arm_prefix}${arm_id}_motor2"><hardwareInterface>franka_hw/FrankaStateInterface</hardwareInterface></actuator>
-      <actuator name="${arm_prefix}${arm_id}_motor3"><hardwareInterface>franka_hw/FrankaStateInterface</hardwareInterface></actuator>
-      <actuator name="${arm_prefix}${arm_id}_motor4"><hardwareInterface>franka_hw/FrankaStateInterface</hardwareInterface></actuator>
-      <actuator name="${arm_prefix}${arm_id}_motor5"><hardwareInterface>franka_hw/FrankaStateInterface</hardwareInterface></actuator>
-      <actuator name="${arm_prefix}${arm_id}_motor6"><hardwareInterface>franka_hw/FrankaStateInterface</hardwareInterface></actuator>
-      <actuator name="${arm_prefix}${arm_id}_motor7"><hardwareInterface>franka_hw/FrankaStateInterface</hardwareInterface></actuator>
+      <joint name="${arm_prefix}_${arm_id}_joint1"><hardwareInterface>franka_hw/FrankaStateInterface</hardwareInterface></joint>
+      <joint name="${arm_prefix}_${arm_id}_joint2"><hardwareInterface>franka_hw/FrankaStateInterface</hardwareInterface></joint>
+      <joint name="${arm_prefix}_${arm_id}_joint3"><hardwareInterface>franka_hw/FrankaStateInterface</hardwareInterface></joint>
+      <joint name="${arm_prefix}_${arm_id}_joint4"><hardwareInterface>franka_hw/FrankaStateInterface</hardwareInterface></joint>
+      <joint name="${arm_prefix}_${arm_id}_joint5"><hardwareInterface>franka_hw/FrankaStateInterface</hardwareInterface></joint>
+      <joint name="${arm_prefix}_${arm_id}_joint6"><hardwareInterface>franka_hw/FrankaStateInterface</hardwareInterface></joint>
+      <joint name="${arm_prefix}_${arm_id}_joint7"><hardwareInterface>franka_hw/FrankaStateInterface</hardwareInterface></joint>
+      <actuator name="${arm_prefix}_${arm_id}_motor1"><hardwareInterface>franka_hw/FrankaStateInterface</hardwareInterface></actuator>
+      <actuator name="${arm_prefix}_${arm_id}_motor2"><hardwareInterface>franka_hw/FrankaStateInterface</hardwareInterface></actuator>
+      <actuator name="${arm_prefix}_${arm_id}_motor3"><hardwareInterface>franka_hw/FrankaStateInterface</hardwareInterface></actuator>
+      <actuator name="${arm_prefix}_${arm_id}_motor4"><hardwareInterface>franka_hw/FrankaStateInterface</hardwareInterface></actuator>
+      <actuator name="${arm_prefix}_${arm_id}_motor5"><hardwareInterface>franka_hw/FrankaStateInterface</hardwareInterface></actuator>
+      <actuator name="${arm_prefix}_${arm_id}_motor6"><hardwareInterface>franka_hw/FrankaStateInterface</hardwareInterface></actuator>
+      <actuator name="${arm_prefix}_${arm_id}_motor7"><hardwareInterface>franka_hw/FrankaStateInterface</hardwareInterface></actuator>
     </transmission>
   </xacro:macro>
@@ -187,5 +187,5 @@
   <!-- ============================================================ -->
   <xacro:macro name="transmission-franka-model" params="arm_id:=fer root:=fer_joint1 tip:=fer_joint7">
-    <transmission name="${arm_prefix}${arm_id}_franka_model">
+    <transmission name="${arm_prefix}_${arm_id}_franka_model">
       <type>franka_hw/FrankaModelInterface</type>
       <joint name="${root}">
