Commit message: modification: aligned FR3 model updates for the dual-arm backup-CBF work
- end_effectors/franka_hand/inertials.yaml: hand/finger inertial values used
  by the aligned dynamics model
- end_effectors/common/utils.xacro, robots/common/utils.xacro,
  mjcf/end_effectors/common/franka_hand.xml.xacro,
  mjcf/robots/common/franka_robot.xml.xacro: xacro updates for the aligned
  MJCF/URDF generation (fix_finger support, consistent wrist/hand lumping)
- .docker & scripts: file-mode normalization

Co-Authored-By: Claude Fable 5 <noreply@anthropic.com>

File: end_effectors/common/utils.xacro (robot description, xacro)
@@ -73,31 +73,16 @@
   <!-- direction: One of { x, y, z, -x, -y, -z }                   -->
   <!-- =========================================================== -->
+  <!-- Single <capsule> primitive (pinocchio/coal parse it directly);
+       historically a cylinder + two cap spheres. -->
   <xacro:macro name="collision_capsule" params="radius length xyz:='0 0 0' direction:='z'">
     <xacro:property name="r" value="${pi/2.0 if 'y' in direction else 0}" />
     <xacro:property name="p" value="${pi/2.0 if 'x' in direction else 0}" />
-    <xacro:property name="y" value="0" />
     <xacro:property name="x" value="${xyz.split(' ')[0]}" />
     <xacro:property name="y" value="${xyz.split(' ')[1]}" />
     <xacro:property name="z" value="${xyz.split(' ')[2]}" />
-    <!-- Sphere center offsets from center of cylinder -->
-    <xacro:property name="sx" value="${length / 2.0 if 'x' in direction else 0}" />
-    <xacro:property name="sy" value="${length / 2.0 if 'y' in direction else 0}" />
-    <xacro:property name="sz" value="${length / 2.0 if 'z' in direction else 0}" />
     <collision>
-      <origin xyz="${x} ${y} ${z}" rpy="${r} ${p} ${y}"/>
+      <origin xyz="${x} ${y} ${z}" rpy="${r} ${p} 0"/>
       <geometry>
-        <cylinder radius="${radius}" length="${length}" />
-      </geometry>
-    </collision>
-    <collision>
-      <origin xyz="${x+sx} ${y+sy} ${z+sz}" />
-      <geometry>
-        <sphere radius="${radius}" />
-      </geometry>
-    </collision>
-    <collision>
-      <origin xyz="${x-sx} ${y-sy} ${z-sz}" />
-      <geometry>
-        <sphere radius="${radius}" />
+        <capsule radius="${radius}" length="${length}" />
       </geometry>
     </collision>

File: mjcf/end_effectors/common/franka_hand.xml.xacro (robot description, xacro)
@@ -12,4 +12,5 @@
                         tcp_rpy:='0 0 0'
                         no_prefix:=false
+                        fix_finger:=false
                         hand_vis_mesh_indices:='[0]'
                         finger_vis_mesh_indices:='[0]'
@@ -31,5 +32,7 @@
             <!-- leftfinger body -->
             <body name="${ee_prefix}leftfinger" pos="0 0 0.0584" euler="0 0 0" gravcomp="1">
-                <joint name="${ee_prefix}finger_joint1" class="finger" />
+                <xacro:unless value="${fix_finger}">
+                    <joint name="${ee_prefix}finger_joint1" class="finger" />
+                </xacro:unless>
                 <xacro:ee-inertial name="leftfinger" />
                 <!-- Visual mesh geoms -->
@@ -44,5 +47,7 @@
             <!-- rightfinger body -->
             <body name="${ee_prefix}rightfinger" pos="0 0 0.0584" euler="0 0 ${pi}" gravcomp="1">
-                <joint name="${ee_prefix}finger_joint2" class="finger" />
+                <xacro:unless value="${fix_finger}">
+                    <joint name="${ee_prefix}finger_joint2" class="finger" />
+                </xacro:unless>
                 <xacro:ee-inertial name="rightfinger" />
                 <!-- Visual mesh geoms -->

File: mjcf/robots/common/franka_robot.xml.xacro (robot description, xacro)
@@ -15,4 +15,5 @@
                          tcp_rpy:='0 0 0'
                          hand:=true
+                         fix_finger:=false
                          ee_id:=none
                          special_connection:=''
@@ -82,4 +83,5 @@
                         tcp_xyz="${tcp_xyz}"
                         tcp_rpy="${tcp_rpy}"
+                        fix_finger="${fix_finger}"
                         hand_vis_mesh_indices="${hand_vis_mesh_indices}"
                         finger_vis_mesh_indices="${finger_vis_mesh_indices}"

File: robots/common/utils.xacro (robot description, xacro)
@@ -67,12 +67,14 @@
   </xacro:macro>
   <!-- =========================================================== -->
-  <!-- Add a <collision> tag with a capsule, made from a cylinder  -->
-  <!-- with two spheres at its caps. The capsule will always be    -->
-  <!-- aligned with the axis of 'direction' you pass along.        -->
+  <!-- Add a <collision> tag with a single <capsule> primitive.    -->
+  <!-- (Historically a cylinder + two cap spheres, because plain   -->
+  <!-- URDF has no capsule element; pinocchio/coal parse <capsule> -->
+  <!-- directly, giving 1/3 the collision pairs and a smooth       -->
+  <!-- distance gradient.)                                         -->
   <!--                                                             -->
-  <!-- radius: Radii of both the cylinder and both spheres [m]     -->
-  <!-- length: Length of the cylinder/distance between the centers -->
-  <!--         of the spheres. NOT overall length of capsule!      -->
-  <!-- xyz:    Position of the center of the capsule/cylinder      -->
+  <!-- radius: Radius of the capsule [m]                           -->
+  <!-- length: Distance between the centers of the cap spheres.    -->
+  <!--         NOT overall length of capsule!                      -->
+  <!-- xyz:    Position of the center of the capsule               -->
   <!-- direction: One of { x, y, z, -x, -y, -z }                   -->
   <!-- =========================================================== -->
@@ -80,28 +82,11 @@
     <xacro:property name="r" value="${pi/2.0 if 'y' in direction else 0}" />
     <xacro:property name="p" value="${pi/2.0 if 'x' in direction else 0}" />
-    <xacro:property name="y" value="0" />
     <xacro:property name="x" value="${xyz.split(' ')[0]}" />
     <xacro:property name="y" value="${xyz.split(' ')[1]}" />
     <xacro:property name="z" value="${xyz.split(' ')[2]}" />
-    <!-- Sphere center offsets from center of cylinder -->
-    <xacro:property name="sx" value="${length / 2.0 if 'x' in direction else 0}" />
-    <xacro:property name="sy" value="${length / 2.0 if 'y' in direction else 0}" />
-    <xacro:property name="sz" value="${length / 2.0 if 'z' in direction else 0}" />
     <collision>
-      <origin xyz="${x} ${y} ${z}" rpy="${r} ${p} ${y}"/>
+      <origin xyz="${x} ${y} ${z}" rpy="${r} ${p} 0"/>
       <geometry>
-        <cylinder radius="${radius}" length="${length}" />
-      </geometry>
-    </collision>
-    <collision>
-      <origin xyz="${x+sx} ${y+sy} ${z+sz}" />
-      <geometry>
-        <sphere radius="${radius}" />
-      </geometry>
-    </collision>
-    <collision>
-      <origin xyz="${x-sx} ${y-sy} ${z-sz}" />
-      <geometry>
-        <sphere radius="${radius}" />
+        <capsule radius="${radius}" length="${length}" />
       </geometry>
     </collision>
