Commit message: add: parameter "use_mujoco" fpr mujoco interface

File: robots/common/franka_arm.ros2_control.xacro (robot description, xacro)
@@ -9,5 +9,6 @@
                  hand:=false
                  gazebo_effort:=false
-                 arm_prefix:=''">
+                 arm_prefix:=''
+                 use_mujoco:=false">
     <xacro:property name="arm_prefix_modified" value="${'' if arm_prefix == '' else arm_prefix + '_'}" />
     <ros2_control name="${arm_prefix_modified}FrankaHardwareInterface" type="system">
@@ -16,4 +17,5 @@
           <param name="arm_id">${arm_id}</param>
           <param name="prefix">${arm_prefix}</param>
+          <param name="load_gripper">${hand}</param>
           <xacro:if value="${use_fake_hardware}">
             <plugin>mock_components/GenericSystem</plugin>
@@ -24,5 +26,8 @@
             <plugin>franka_gz_ros2_control/GZSystem</plugin>
           </xacro:if>
-          <xacro:if value="${use_fake_hardware == 0 and gazebo == 0}">
+          <xacro:if value="${use_mujoco}">
+            <plugin>franka_mujoco/FrankaMujocoSystem</plugin>
+          </xacro:if>
+          <xacro:if value="${use_fake_hardware == 0 and gazebo == 0 and use_mujoco == 0}">
             <plugin>franka_hardware/FrankaHardwareInterface</plugin>
             <param name="robot_ip">${robot_ip}</param>
@@ -37,6 +42,6 @@
             https://github.com/ros-controls/gz_ros2_control/issues/343
             Command Interfaces -->
-            <command_interface name="position"/>
-            <command_interface name="velocity"/>
+          <command_interface name="position"/>
+          <command_interface name="velocity"/>
           <xacro:if value="${gazebo == 0 or gazebo_effort == 1}">
             <command_interface name="effort"/>
@@ -61,28 +66,30 @@
         <xacro:configure_joint joint_name="${arm_prefix_modified}${arm_id}_finger_joint1" initial_position="0.0" />
       </xacro:if>
-      <xacro:macro name="general_purpose_io" params="prefix command_interface index">
-        <gpio name="${prefix}">
-          <command_interface name="${command_interface}"/>
-          <param name="index">${index}</param>
-        </gpio>
-      </xacro:macro>
-      <!-- Cartesian velocity interfaces -->
-      <xacro:general_purpose_io prefix="${arm_prefix_modified}vx" command_interface="cartesian_velocity" index="0"/>
-      <xacro:general_purpose_io prefix="${arm_prefix_modified}vy" command_interface="cartesian_velocity" index="1"/>
-      <xacro:general_purpose_io prefix="${arm_prefix_modified}vz" command_interface="cartesian_velocity" index="2"/>
-      <xacro:general_purpose_io prefix="${arm_prefix_modified}wx" command_interface="cartesian_velocity" index="3"/>
-      <xacro:general_purpose_io prefix="${arm_prefix_modified}wy" command_interface="cartesian_velocity" index="4"/>
-      <xacro:general_purpose_io prefix="${arm_prefix_modified}wz" command_interface="cartesian_velocity" index="5"/>
-      <!-- Cartesian pose interfaces, in total 16 interfaces -->
-      <xacro:macro name="loop" params="i">
-        <xacro:unless value="${i == 16}">
-          <xacro:general_purpose_io prefix="${arm_prefix_modified}${i}" command_interface="cartesian_pose_command" index="${i}"/>
-          <xacro:loop i="${i+1}"/>
-        </xacro:unless>
-      </xacro:macro>
-      <xacro:loop i="0"/>
-      <!-- Elbow command interfaces -->
-      <xacro:general_purpose_io prefix="${arm_prefix_modified}joint_3_position" command_interface="elbow_command" index="0"/>
-      <xacro:general_purpose_io prefix="${arm_prefix_modified}joint_4_sign" command_interface="elbow_command" index="1"/>
+      <xacro:unless value="${use_mujoco}">
+        <xacro:macro name="general_purpose_io" params="prefix command_interface index">
+          <gpio name="${prefix}">
+            <command_interface name="${command_interface}"/>
+            <param name="index">${index}</param>
+          </gpio>
+        </xacro:macro>
+        <!-- Cartesian velocity interfaces -->
+        <xacro:general_purpose_io prefix="${arm_prefix_modified}vx" command_interface="cartesian_velocity" index="0"/>
+        <xacro:general_purpose_io prefix="${arm_prefix_modified}vy" command_interface="cartesian_velocity" index="1"/>
+        <xacro:general_purpose_io prefix="${arm_prefix_modified}vz" command_interface="cartesian_velocity" index="2"/>
+        <xacro:general_purpose_io prefix="${arm_prefix_modified}wx" command_interface="cartesian_velocity" index="3"/>
+        <xacro:general_purpose_io prefix="${arm_prefix_modified}wy" command_interface="cartesian_velocity" index="4"/>
+        <xacro:general_purpose_io prefix="${arm_prefix_modified}wz" command_interface="cartesian_velocity" index="5"/>
+        <!-- Cartesian pose interfaces, in total 16 interfaces -->
+        <xacro:macro name="loop" params="i">
+          <xacro:unless value="${i == 16}">
+            <xacro:general_purpose_io prefix="${arm_prefix_modified}${i}" command_interface="cartesian_pose_command" index="${i}"/>
+            <xacro:loop i="${i+1}"/>
+          </xacro:unless>
+        </xacro:macro>
+        <xacro:loop i="0"/>
+        <!-- Elbow command interfaces -->
+        <xacro:general_purpose_io prefix="${arm_prefix_modified}joint_3_position" command_interface="elbow_command" index="0"/>
+        <xacro:general_purpose_io prefix="${arm_prefix_modified}joint_4_sign" command_interface="elbow_command" index="1"/>
+      </xacro:unless>
     </ros2_control>
     <xacro:if value="${gazebo}">

File: robots/common/franka_robot.xacro (robot description, xacro)
@@ -22,4 +22,5 @@
                       with_sc:='false'
                       ros2_control:=false
+                      use_mujoco:=false
                       robot_ip:=''
                       use_fake_hardware:=false
@@ -155,4 +156,5 @@
           gazebo_effort="${gazebo_effort}"
           arm_prefix="${arm_prefix}"
+          use_mujoco="${use_mujoco}"
       />
     </xacro:if>

File: robots/fr3/fr3.urdf.xacro (robot description, xacro)
@@ -14,4 +14,5 @@
   <!-- Should an end-effector be mounted at the flange?" -->
   <xacro:arg name="hand" default="true" />
+  <xacro:arg name="fix_finger" default="false" />
   <!-- Which end-effector would be mounted at the flange?" -->
   <xacro:arg name="ee_id" default="franka_hand" />
@@ -32,4 +33,5 @@
   <!-- Is the robot being controlled with ros2_control?" -->
   <xacro:arg name="ros2_control" default="false" />
+  <xacro:arg name="use_mujoco" default="false" />
   <!-- IP address or hostname of the robot" -->
   <xacro:arg name="robot_ip" default="" />
@@ -64,4 +66,5 @@
                       with_sc="$(arg with_sc)"
                       ros2_control="$(arg ros2_control)"
+                      use_mujoco="$(arg use_mujoco)"
                       robot_ip="$(arg robot_ip)"
                       use_fake_hardware="$(arg use_fake_hardware)"
@@ -71,5 +74,6 @@
                       arm_prefix="${modified_prefix}"
                       description_pkg="$(arg description_pkg)"
-                      connected_to= "base">
+                      connected_to= "base"
+                      fix_finger="$(arg fix_finger)">
   </xacro:franka_robot>
 </robot>
