Commit message: fix: errors for MJCF

File: mjcf/end_effectors/common/ee_with_one_link.xml.xacro (robot description, xacro)
@@ -1,4 +1,5 @@
 <?xml version="1.0" encoding="utf-8"?>
 <mujoco xmlns:xacro="http://www.ros.org/wiki/xacro">
+    <xacro:include filename="utils.xml.xacro" />
     <xacro:macro name="ee_with_one_link"
                 params="arm_id arm_prefix:=''

File: mjcf/end_effectors/common/franka_hand.xml.xacro (robot description, xacro)
@@ -1,4 +1,5 @@
 <?xml version="1.0" encoding="utf-8"?>
 <mujoco xmlns:xacro="http://www.ros.org/wiki/xacro">
+    <xacro:include filename="utils.xml.xacro" />
     <!-- Caution: 'connected_to' do not adapt to MuJoCo, this macro have to put correctly under desired "connected" body -->
     <xacro:macro name="franka_hand"
@@ -20,4 +21,6 @@
             <xacro:property name="ee_prefix" value="${arm_prefix_modified}${arm_id}_" />
         </xacro:unless>
+        <xacro:property name="finger_vis_indices_raw" value="${str(finger_vis_mesh_indices).strip('[]')}" />
+        <xacro:property name="finger_vis_materials_raw" value="${str(finger_vis_mesh_materials).strip('[]')}" />
         <!--  hand body  -->
         <body name="${ee_prefix}hand" pos="${xyz_ee}" euler="${rpy_ee}">
@@ -30,7 +33,5 @@
                 <xacro:ee-inertial name="leftfinger" />
                 <!-- Visual mesh geoms -->
-                <xacro:for value="idx" in="${finger_vis_mesh_indices}">
-                    <geom name="${ee_prefix}leftfinger_${idx}_visual" type="mesh" mesh="finger_${idx}" material="${finger_vis_mesh_materials[idx] if finger_vis_mesh_materials else 'white'}" class="visual" />
-                </xacro:for>
+                <xacro:emit_ee_visual_meshes geom_prefix="${ee_prefix}" geom_name_stem="leftfinger" mesh_name_stem="finger" vis_indices_raw="${finger_vis_indices_raw}" vis_materials_raw="${finger_vis_materials_raw}" i="0" />
                 <!-- Collision geoms -->
                 <geom type="box" size="0.0085 0.004 0.0085" pos="0 0.0055 0.0445"/>
@@ -45,7 +46,5 @@
                 <xacro:ee-inertial name="rightfinger" />
                 <!-- Visual mesh geoms -->
-                <xacro:for value="idx" in="${finger_vis_mesh_indices}">
-                    <geom name="${ee_prefix}rightfinger_${idx}_visual" type="mesh" mesh="finger_${idx}" material="${finger_vis_mesh_materials[idx] if finger_vis_mesh_materials else 'white'}" class="visual" />
-                </xacro:for>
+                <xacro:emit_ee_visual_meshes geom_prefix="${ee_prefix}" geom_name_stem="rightfinger" mesh_name_stem="finger" vis_indices_raw="${finger_vis_indices_raw}" vis_materials_raw="${finger_vis_materials_raw}" i="0" />
                 <!-- Collision geoms -->
                 <geom type="box" size="0.0085 0.004 0.0085" pos="0 0.0055 0.0445"/>

File: mjcf/end_effectors/common/utils.xml.xacro (robot description, xacro)
@@ -29,9 +29,25 @@
     <!-- vis_mesh_indices:   List of visual sub-mesh indices        -->
     <!-- ========================================================== -->
+    <!-- Recursive helper to emit visual meshes without xacro:for (not available in Humble) -->
+    <xacro:macro name="emit_ee_visual_meshes" params="geom_prefix geom_name_stem mesh_name_stem vis_indices_raw vis_materials_raw i">
+        <xacro:unless value="${str(vis_indices_raw) == '' or i == len(str(vis_indices_raw).split(','))}">
+            <xacro:property name="idx" value="${str(vis_indices_raw).split(',')[i].strip()}" />
+            <xacro:property name="mat_raw"
+                            value="${(str(vis_materials_raw).split(',')[i].strip().strip(&quot;'&quot;))
+                                    if (str(vis_materials_raw).strip() != '' and i &lt; len(str(vis_materials_raw).split(',')))
+                                    else ''}" />
+            <geom name="${geom_prefix}${geom_name_stem}_${idx}_visual"
+                  type="mesh"
+                  mesh="${mesh_name_stem}_${idx}"
+                  material="${mat_raw if mat_raw != '' else 'white'}"
+                  class="visual" />
+            <xacro:emit_ee_visual_meshes geom_prefix="${geom_prefix}" geom_name_stem="${geom_name_stem}" mesh_name_stem="${mesh_name_stem}" vis_indices_raw="${vis_indices_raw}" vis_materials_raw="${vis_materials_raw}" i="${i+1}" />
+        </xacro:unless>
+    </xacro:macro>
     <xacro:macro name="ee_link_with_sc" params="name prefix:=${ee_prefix} vis_mesh_indices:='[0]' vis_mesh_materials:='['']'">
-        <!-- Visual mesh geoms: one geom per sub-mesh index -->
-        <xacro:for value="idx" in="${vis_mesh_indices}">
-            <geom name="${prefix}${name}_${idx}_visual" type="mesh" mesh="${name}_${idx}" material="${vis_mesh_materials[idx] if vis_mesh_materials else 'white'}" class="visual" />
-        </xacro:for>
+        <!-- Visual mesh geoms: expand indices with recursion -->
+        <xacro:property name="vis_indices_raw" value="${str(vis_mesh_indices).strip('[]')}" />
+        <xacro:property name="vis_materials_raw" value="${str(vis_mesh_materials).strip('[]')}" />
+        <xacro:emit_ee_visual_meshes geom_prefix="${prefix}" geom_name_stem="${name}" mesh_name_stem="${name}" vis_indices_raw="${vis_indices_raw}" vis_materials_raw="${vis_materials_raw}" i="0" />
         <!-- Collision mesh geom: single mesh named {name}_coll -->
         <geom name="${prefix}${name}_coll_collision" type="mesh" mesh="${name}_coll" class="collision" />

File: mjcf/robots/common/franka_robot.xml.xacro (robot description, xacro)
@@ -20,5 +20,4 @@
                          arm_prefix:=''
                          connected_to:='base'
-                         fix_finger:=false
                          link0_vis_mesh_indices:='[0]'
                          link1_vis_mesh_indices:='[0]'
@@ -42,5 +41,5 @@
                          hand_vis_mesh_materials:='[]'
                          finger_vis_mesh_materials:='[]'
-                         ee_vis_mesh_materials">
+                         ee_vis_mesh_materials:='[]'">
         <xacro:franka_arm
             arm_id="${arm_id}"
@@ -77,10 +76,9 @@
                         arm_prefix="${arm_prefix}"
                         no_prefix="${no_prefix}"
-                        ee_inertials="${xacro.load_yaml('$(find franka_description)/end_effectors/' + ee_id + '/inertials.yaml')}"
+                        ee_inertials="${xacro.load_yaml('$(find franka_description)/mjcf/end_effectors/' + ee_id + '/inertials.yaml')}"
                         xyz_ee="${xyz_ee}"
                         rpy_ee="${rpy_ee}"
                         tcp_xyz="${tcp_xyz}"
                         tcp_rpy="${tcp_rpy}"
-                        fix_finger="${fix_finger}"
                         hand_vis_mesh_indices="${hand_vis_mesh_indices}"
                         finger_vis_mesh_indices="${finger_vis_mesh_indices}"
@@ -94,5 +92,5 @@
                         arm_prefix="${arm_prefix}"
                         ee_id="${ee_id}"
-                        ee_inertials="${xacro.load_yaml('$(find franka_description)/end_effectors/' + ee_id + '/inertials.yaml')}"
+                        ee_inertials="${xacro.load_yaml('$(find franka_description)/mjcf/end_effectors/' + ee_id + '/inertials.yaml')}"
                         xyz_ee="${xyz_ee}"
                         rpy_ee="${rpy_ee}"

File: mjcf/robots/common/utils.xml.xacro (robot description, xacro)
@@ -29,10 +29,26 @@
     <!-- with_accelerometers: Include accelerometer sites           -->
     <!-- ========================================================== -->
+    <!-- Recursive helper to emit visual meshes without xacro:for (not available in Humble) -->
+    <xacro:macro name="emit_visual_meshes" params="prefix name vis_indices_raw vis_materials_raw i">
+        <xacro:unless value="${str(vis_indices_raw) == '' or i == len(str(vis_indices_raw).split(','))}">
+            <xacro:property name="idx" value="${str(vis_indices_raw).split(',')[i].strip()}" />
+            <xacro:property name="mat_raw"
+                            value="${(str(vis_materials_raw).split(',')[i].strip().strip(&quot;'&quot;))
+                                    if (str(vis_materials_raw).strip() != '' and i &lt; len(str(vis_materials_raw).split(',')))
+                                    else ''}" />
+            <geom name="${prefix}${name}_${idx}_visual"
+                  material="${mat_raw if mat_raw != '' else 'white'}"
+                  type="mesh"
+                  mesh="${name}_${idx}"
+                  class="visual" />
+            <xacro:emit_visual_meshes prefix="${prefix}" name="${name}" vis_indices_raw="${vis_indices_raw}" vis_materials_raw="${vis_materials_raw}" i="${i+1}" />
+        </xacro:unless>
+    </xacro:macro>
     <xacro:macro name="link_with_sc" params="name no_prefix:='false' vis_mesh_indices:='[]' vis_mesh_materials:='['']' with_accelerometers:=false">
         <xacro:property name="prefix" value="${'' if no_prefix else (arm_id + '_' if arm_prefix == '' else arm_prefix + '_' + arm_id + '_')}" />
-        <!-- Visual mesh geoms: one geom per sub-mesh index -->
-        <xacro:for value="idx" in="${vis_mesh_indices}">
-            <geom name="${prefix}${name}_${idx}_visual" material="${vis_mesh_materials[idx] if vis_mesh_materials else 'white'}" type="mesh" mesh="${name}_${idx}" class="visual" />
-        </xacro:for>
+        <!-- Visual mesh geoms: expand indices with recursion -->
+        <xacro:property name="vis_indices_raw" value="${str(vis_mesh_indices).strip('[]')}" />
+        <xacro:property name="vis_materials_raw" value="${str(vis_mesh_materials).strip('[]')}" />
+        <xacro:emit_visual_meshes prefix="${prefix}" name="${name}" vis_indices_raw="${vis_indices_raw}" vis_materials_raw="${vis_materials_raw}" i="0" />
         <!-- Collision mesh geom: single mesh named {name}_coll -->
         <geom name="${prefix}${name}_collision" type="mesh" mesh="${name}_coll" class="collision" />
@@ -53,8 +69,8 @@
     <xacro:macro name="franka-limits" params="config name">
         <xacro:property name="limits" value="${config[name]['limit']}" lazy_eval="false" />
-        <xacro:property name="franka_lower_${name}"   value="${limits.lower}"    />
-        <xacro:property name="franka_upper_${name}"   value="${limits.upper}"    />
-        <xacro:property name="franka_effort_${name}"  value="${limits.effort}"   />
-        <xacro:property name="franka_velocity_${name}" value="${limits.velocity}" />
+        <xacro:property name="franka_lower_${name}"   value="${limits.lower}"    scope="parent" />
+        <xacro:property name="franka_upper_${name}"   value="${limits.upper}"    scope="parent" />
+        <xacro:property name="franka_effort_${name}"  value="${limits.effort}"   scope="parent" />
+        <xacro:property name="franka_velocity_${name}" value="${limits.velocity}" scope="parent" />
     </xacro:macro>
     <!-- ========================================================================= -->
@@ -67,6 +83,6 @@
     <xacro:macro name="franka-dynamics" params="config name">
         <xacro:property name="dynamics" value="${config[name]['dynamic']}" lazy_eval="false" />
-        <xacro:property name="franka_damping_${name}"  value="${dynamics.damping}"  />
-        <xacro:property name="franka_friction_${name}" value="${dynamics.friction}" />
+        <xacro:property name="franka_damping_${name}"  value="${dynamics.damping}"  scope="parent" />
+        <xacro:property name="franka_friction_${name}" value="${dynamics.friction}" scope="parent" />
     </xacro:macro>
     <!-- ========================================================================= -->
@@ -79,6 +95,6 @@
     <xacro:macro name="franka-kinematics" params="config name">
         <xacro:property name="kinematics" value="${config[name]['kinematic']}" lazy_eval="false" />
-        <xacro:property name="franka_kin_pos_${name}"   value="${kinematics.x} ${kinematics.y} ${kinematics.z}"             />
-        <xacro:property name="franka_kin_euler_${name}" value="${kinematics.roll} ${kinematics.pitch} ${kinematics.yaw}"    />
+        <xacro:property name="franka_kin_pos_${name}"   value="${kinematics.x} ${kinematics.y} ${kinematics.z}"             scope="parent" />
+        <xacro:property name="franka_kin_euler_${name}" value="${kinematics.roll} ${kinematics.pitch} ${kinematics.yaw}"    scope="parent" />
     </xacro:macro>
     <!-- ================================================================================== -->

File: mjcf/robots/fr3/fr3.xml.xacro (robot description, xacro)
@@ -7,5 +7,8 @@
     <!-- ── xacro includes ── -->
     <xacro:include filename="$(find franka_description)/mjcf/robots/common/franka_robot.xml.xacro" />
+    <xacro:include filename="$(find franka_description)/mjcf/robots/common/franka_arm.xml.xacro" />
     <xacro:include filename="$(find franka_description)/mjcf/robots/common/franka_arm_actuator.xml.xacro" />
+    <xacro:include filename="$(find franka_description)/mjcf/end_effectors/common/franka_hand.xml.xacro" />
+    <xacro:include filename="$(find franka_description)/mjcf/end_effectors/common/ee_with_one_link.xml.xacro" />
     <xacro:include filename="$(find franka_description)/mjcf/end_effectors/common/franka_hand_actuator.xml.xacro" />
     <!-- ── xacro args (overridable at parse time) ── -->
@@ -40,7 +43,7 @@
         <global azimuth="150" elevation="-20" />
     </visual>
-    <!-- ── Default classes (레퍼런스 MJCF와 동일) ── -->
+    <!-- Default classes -->
     <default>
-        <default class="${arg arm_id}">
+        <default class="$(arg arm_id)">
             <joint armature="0.1" damping="1"/>
             <position inheritrange="1"/>
@@ -81,6 +84,6 @@
         <mesh name="link0_5" file="robot_arms/fr3/visual/link0_5.obj"/>
         <mesh name="link0_6" file="robot_arms/fr3/visual/link0_6.obj"/>
-        <mesh name="link1_0" file="robot_arms/fr3/visual/link1_0.obj"/>
-        <mesh name="link2_0" file="robot_arms/fr3/visual/link2_0.obj"/>
+        <mesh name="link1_0" file="robot_arms/fr3/visual/link1.obj"/>
+        <mesh name="link2_0" file="robot_arms/fr3/visual/link2.obj"/>
         <mesh name="link3_0" file="robot_arms/fr3/visual/link3_0.obj"/>
         <mesh name="link3_1" file="robot_arms/fr3/visual/link3_1.obj"/>
@@ -112,13 +115,13 @@
         <mesh name="link7_coll" file="robot_arms/fr3/collision/link7.stl"/>
         <!-- hand visual meshes -->
-        <mesh name="hand_0"   file="robot_ee/franka_hand/visual/hand_0.obj"/>
-        <mesh name="hand_1"   file="robot_ee/franka_hand/visual/hand_1.obj"/>
-        <mesh name="hand_2"   file="robot_ee/franka_hand/visual/hand_2.obj"/>
-        <mesh name="hand_3"   file="robot_ee/franka_hand/visual/hand_3.obj"/>
-        <mesh name="hand_4"   file="robot_ee/franka_hand/visual/hand_4.obj"/>
-        <mesh name="finger_0" file="robot_ee/franka_hand/visual/finger_0.obj"/>
-        <mesh name="finger_1" file="robot_ee/franka_hand/visual/finger_1.obj"/>
+        <mesh name="hand_0"   file="robot_ee/franka_hand_white/visual/hand_0.obj"/>
+        <mesh name="hand_1"   file="robot_ee/franka_hand_white/visual/hand_1.obj"/>
+        <mesh name="hand_2"   file="robot_ee/franka_hand_white/visual/hand_2.obj"/>
+        <mesh name="hand_3"   file="robot_ee/franka_hand_white/visual/hand_3.obj"/>
+        <mesh name="hand_4"   file="robot_ee/franka_hand_white/visual/hand_4.obj"/>
+        <mesh name="finger_0" file="robot_ee/franka_hand_white/visual/finger_0.obj"/>
+        <mesh name="finger_1" file="robot_ee/franka_hand_white/visual/finger_1.obj"/>
         <!-- hand collision meshes -->
-        <mesh name="hand_coll" file="robot_ee/franka_hand/collision/hand.stl"/>
+        <mesh name="hand_coll" file="robot_ee/franka_hand_white/collision/hand.stl"/>
     </asset>
     <!-- ── Worldbody ── -->

File: robots/common/franka_arm.ros2_control.xacro (robot description, xacro)
@@ -10,5 +10,15 @@
                  gazebo_effort:=false
                  arm_prefix:=''
-                 use_mujoco:=false">
+                 no_prefix:='false'
+                 use_mujoco:=false
+                 connected_to:='base'
+                 xyz:='0 0 0'
+                 rpy:='0 0 0'
+                 ee_id:=none
+                 xyz_ee:='0 0 0'
+                 rpy_ee:='0 0 0'
+                 tcp_xyz:='0 0 0'
+                 tcp_rpy:='0 0 0'
+                 mujoco_scene_xacro_path:=''">
     <xacro:property name="arm_prefix_modified" value="${'' if arm_prefix == '' else arm_prefix + '_'}" />
     <ros2_control name="${arm_prefix_modified}FrankaHardwareInterface" type="system">
@@ -28,4 +38,18 @@
           <xacro:if value="${use_mujoco}">
             <plugin>franka_mujoco/FrankaMujocoSystem</plugin>
+            <param name="mujoco_scene_xacro_path">$(arg mujoco_scene_xacro_path)</param>
+            <param name="enable_viewer">true</param>
+            <param name="arm_id">${arm_id}</param>
+            <param name="arm_prefix">${arm_prefix}</param>
+            <param name="no_prefix">${no_prefix}</param>
+            <param name="connected_to">${connected_to}</param>
+            <param name="xyz">${xyz}</param>
+            <param name="rpy">${rpy}</param>
+            <param name="hand">${hand}</param>
+            <param name="ee_id">${ee_id}</param>
+            <param name="xyz_ee">${xyz_ee}</param>
+            <param name="rpy_ee">${rpy_ee}</param>
+            <param name="tcp_xyz">${tcp_xyz}</param>
+            <param name="tcp_rpy">${tcp_rpy}</param>
           </xacro:if>
           <xacro:if value="${use_fake_hardware == 0 and gazebo == 0 and use_mujoco == 0}">
@@ -38,19 +62,20 @@
       <xacro:macro name="configure_joint" params="joint_name initial_position">
         <joint name="${joint_name}">
-          <!--
-            deactivated for gazebo velocity and position interface due to a bug
+            <!--
+              deactivated for gazebo velocity and position interface due to a bug
             https://github.com/ros-controls/gz_ros2_control/issues/343
             Command Interfaces -->
-          <command_interface name="position"/>
-          <command_interface name="velocity"/>
-          <xacro:if value="${gazebo == 0 or gazebo_effort == 1}">
-            <command_interface name="effort"/>
-          </xacro:if>
+            <command_interface name="position"/>
+            <command_interface name="velocity"/>
+            <xacro:if value="${gazebo == 0 or gazebo_effort == 1}">
+              <command_interface name="effort"/>
+            </xacro:if>
           <!-- State Interfaces -->
           <state_interface name="position">
             <param name="initial_value">${initial_position}</param>
           </state_interface>
-          <state_interface name="velocity"/>
+          <state_interface name="velocity">
             <param name="initial_value">0.0</param>
+          </state_interface>
           <state_interface name="effort"/>
         </joint>

File: robots/common/franka_robot.xacro (robot description, xacro)
@@ -23,4 +23,5 @@
                       ros2_control:=false
                       use_mujoco:=false
+                      mujoco_scene_xacro_path:=''
                       robot_ip:=''
                       use_fake_hardware:=false
@@ -157,4 +158,13 @@
           arm_prefix="${arm_prefix}"
           use_mujoco="${use_mujoco}"
+          no_prefix="${no_prefix}"
+          connected_to="${connected_to}"
+          xyz="${xyz}"
+          rpy="${rpy}"
+          ee_id="${ee_id}"
+          xyz_ee="${xyz_ee}"
+          rpy_ee="${rpy_ee}"
+          tcp_xyz="${tcp_xyz}"
+          tcp_rpy="${tcp_rpy}"
       />
     </xacro:if>

File: robots/fr3/fr3.urdf.xacro (robot description, xacro)
@@ -34,4 +34,6 @@
   <xacro:arg name="ros2_control" default="false" />
   <xacro:arg name="use_mujoco" default="false" />
+  <!-- MuJoCo scene XML string (generated from mujoco_scene_xacro in the launch file) -->
+  <xacro:arg name="mujoco_scene_xacro_path" default="" />
   <!-- IP address or hostname of the robot" -->
   <xacro:arg name="robot_ip" default="" />
@@ -67,4 +69,5 @@
                       ros2_control="$(arg ros2_control)"
                       use_mujoco="$(arg use_mujoco)"
+                      mujoco_scene_xacro_path="$(arg mujoco_scene_xacro_path)"
                       robot_ip="$(arg robot_ip)"
                       use_fake_hardware="$(arg use_fake_hardware)"
