Commit message: update ert mujoco_ros_hardware

File: mjcf/end_effectors/common/franka_hand_actuator.xml.xacro (robot description, xacro)
@@ -8,5 +8,5 @@
         </xacro:unless>
         <tendon>
-            <fixed name="finger">
+            <fixed name="${ee_prefix}finger">
             <joint joint="${ee_prefix}finger_joint1" coef="0.5"/>
             <joint joint="${ee_prefix}finger_joint2" coef="0.5"/>
@@ -17,5 +17,5 @@
         </equality>
         <actuator>
-            <general class="${arm_id}" name="${ee_prefix}hand" tendon="finger" forcerange="-100 100" ctrlrange="0 255" gainprm="0.01568627451 0 0" biasprm="0 -100 -10"/>
+            <general class="${arm_id}" name="${ee_prefix}hand" tendon="${ee_prefix}finger" forcerange="-100 100" ctrlrange="0 255" gainprm="0.01568627451 0 0" biasprm="0 -100 -10"/>
         </actuator>
     </xacro:macro>

File: mjcf/robots/fr3/fr3.xml.xacro (robot description, xacro)
@@ -1,8 +1,4 @@
 <?xml version="1.0" encoding="utf-8"?>
 <mujoco xmlns:xacro="http://www.ros.org/wiki/xacro" model="fr3">
-    <!-- ================================================================ -->
-    <!--  fr3.xml.xacro                                                    -->
-    <!--  FR3 로봇의 최상위 MuJoCo 파일.                                    -->
-    <!-- ================================================================ -->
     <!-- ── xacro includes ── -->
     <xacro:include filename="$(find franka_description)/mjcf/robots/common/franka_robot.xml.xacro" />
@@ -21,6 +17,6 @@
     <xacro:arg name="hand"           default="true" />
     <xacro:arg name="ee_id"          default="franka_hand" />
-    <xacro:arg name="xyz_ee"         default="0 0 0.107" />
-    <xacro:arg name="rpy_ee"         default="0 0 -0.7853981633974483" />
+    <xacro:arg name="xyz_ee"         default="0 0 0" />
+    <xacro:arg name="rpy_ee"         default="0 0 ${-pi/4}" />
     <xacro:arg name="tcp_xyz"        default="0 0 0.1034" />
     <xacro:arg name="tcp_rpy"        default="0 0 0" />

File: robots/common/franka_arm.ros2_control.xacro (robot description, xacro)
@@ -11,14 +11,5 @@
                  arm_prefix:=''
                  no_prefix:='false'
-                 use_mujoco:=false
-                 connected_to:='base'
-                 xyz:='0 0 0'
-                 rpy:='0 0 0'
-                 ee_id:=none
-                 xyz_ee:='0 0 0'
-                 rpy_ee:='0 0 0'
-                 tcp_xyz:='0 0 0'
-                 tcp_rpy:='0 0 0'
-                 mujoco_scene_xacro_path:=''">
+                 use_mujoco:=false">
     <xacro:property name="arm_prefix_modified" value="${'' if arm_prefix == '' else arm_prefix + '_'}" />
     <ros2_control name="${arm_prefix_modified}FrankaHardwareInterface" type="system">
@@ -37,19 +28,6 @@
           </xacro:if>
           <xacro:if value="${use_mujoco}">
-            <plugin>franka_mujoco/FrankaMujocoSystem</plugin>
-            <param name="mujoco_scene_xacro_path">$(arg mujoco_scene_xacro_path)</param>
-            <param name="enable_viewer">true</param>
-            <param name="arm_id">${arm_id}</param>
-            <param name="arm_prefix">${arm_prefix}</param>
-            <param name="no_prefix">${no_prefix}</param>
-            <param name="connected_to">${connected_to}</param>
-            <param name="xyz">${xyz}</param>
-            <param name="rpy">${rpy}</param>
-            <param name="hand">${hand}</param>
-            <param name="ee_id">${ee_id}</param>
-            <param name="xyz_ee">${xyz_ee}</param>
-            <param name="rpy_ee">${rpy_ee}</param>
-            <param name="tcp_xyz">${tcp_xyz}</param>
-            <param name="tcp_rpy">${tcp_rpy}</param>
+            <plugin>mujoco_ros_hardware/MujocoHardwareInterface</plugin>
+            <param name="robot_type">franka</param>
           </xacro:if>
           <xacro:if value="${use_fake_hardware == 0 and gazebo == 0 and use_mujoco == 0}">

File: robots/common/franka_multi_arm.ros2_control.xacro (robot description, xacro)
@@ -3,5 +3,5 @@
 <xacro:macro name="franka_multi_arm_ros2_control"
          params="arm_ids
-                 robot_ips
+                 robot_ips:=''
                  robot_prefixes:=''
                  use_fake_hardware:=false
@@ -9,10 +9,20 @@
                  gazebo:=false
                  hand:=false
-                 gazebo_effort:=false">
+                 gazebo_effort:=false
+                 use_mujoco:=false
+                 mujoco_scene_xacro_path:=''
+                 xyzs:='0 0 0'
+                 rpys:='0 0 0'
+                 connected_to:='base'
+                 ee_id:=none
+                 xyz_ee:='0 0 0'
+                 rpy_ee:='0 0 0'
+                 tcp_xyz:='0 0 0'
+                 tcp_rpy:='0 0 0'">
     <!-- arm_ids/robot_ips/robot_prefixes accept comma or space separated values. -->
     <xacro:property name="arm_ids_list"
                     value="${[x.strip() for x in (arm_ids.split(',') if ',' in arm_ids else arm_ids.split()) if x.strip() != '']}" />
     <xacro:property name="robot_ips_list"
-                    value="${[x.strip() for x in (robot_ips.split(',') if ',' in robot_ips else robot_ips.split()) if x.strip() != '']}" />
+                    value="${[x.strip() for x in (robot_ips.split(',') if ',' in robot_ips else robot_ips.split()) if x.strip() != ''] if robot_ips != '' else []}" />
     <xacro:property name="robot_prefixes_raw"
                     value="${[x.strip() for x in (robot_prefixes.split(',') if ',' in robot_prefixes else robot_prefixes.split()) if x.strip() != '']}" />
@@ -20,8 +30,14 @@
                     value="${(['' for _ in range(len(arm_ids_list))] if len(robot_prefixes_raw) == 0 else ['' if p in ['','none','null'] else p for p in robot_prefixes_raw])}" />
     <xacro:property name="robot_count" value="${len(arm_ids_list)}" />
+    <!-- xyzs/rpys: semicolon-separated, one entry per arm -->
+    <xacro:property name="xyz_list"
+                    value="${[x.strip() for x in xyzs.split(';') if x.strip() != '']}" />
+    <xacro:property name="rpy_list"
+                    value="${[x.strip() for x in rpys.split(';') if x.strip() != '']}" />
+    <!-- real-hardware param loop (arm_id, robot_ip, prefix) -->
     <xacro:macro name="robot_param_loop" params="i">
       <xacro:unless value="${i == robot_count}">
         <xacro:property name="arm_id_i" value="${arm_ids_list[i]}" />
-        <xacro:property name="robot_ip_i" value="${robot_ips_list[i]}" />
+        <xacro:property name="robot_ip_i" value="${robot_ips_list[i] if i &lt; len(robot_ips_list) else ''}" />
         <xacro:property name="robot_prefix_i"
                         value="${robot_prefixes_list[i] if i &lt; len(robot_prefixes_list) else ''}" />
@@ -32,4 +48,16 @@
         </xacro:if>
         <xacro:robot_param_loop i="${i+1}"/>
+      </xacro:unless>
+    </xacro:macro>
+    <!-- mujoco param loop — outputs hw_params expected by FrankaMultiSubHandler:
+         arm_id_<i>, prefix_<i>, load_gripper_<i> -->
+    <xacro:macro name="mujoco_param_loop" params="i">
+      <xacro:unless value="${i == robot_count}">
+        <xacro:property name="arm_id_i"       value="${arm_ids_list[i]}" />
+        <xacro:property name="robot_prefix_i" value="${robot_prefixes_list[i] if i &lt; len(robot_prefixes_list) else ''}" />
+        <param name="arm_id_${i}">${arm_id_i}</param>
+        <param name="prefix_${i}">${robot_prefix_i}</param>
+        <param name="load_gripper_${i}">${hand}</param>
+        <xacro:mujoco_param_loop i="${i+1}"/>
       </xacro:unless>
     </xacro:macro>
@@ -46,8 +74,14 @@
             <plugin>franka_gz_ros2_control/GZSystem</plugin>
           </xacro:if>
-          <xacro:if value="${use_fake_hardware == 0 and gazebo == 0}">
+          <xacro:if value="${use_mujoco}">
+            <plugin>mujoco_ros_hardware/MujocoHardwareInterface</plugin>
+            <param name="robot_type">franka_multi</param>
+            <param name="robot_count">${robot_count}</param>
+            <xacro:mujoco_param_loop i="0"/>
+          </xacro:if>
+          <xacro:if value="${use_fake_hardware == 0 and gazebo == 0 and use_mujoco == 0}">
             <plugin>franka_hardware/FrankaMultiHardwareInterface</plugin>
+            <xacro:robot_param_loop i="0"/>
           </xacro:if>
-          <xacro:robot_param_loop i="0"/>
         </hardware>
       <!-- Joint position, velocity and effort interfaces -->
@@ -67,6 +101,7 @@
             <param name="initial_value">${initial_position}</param>
           </state_interface>
-          <state_interface name="velocity"/>
+          <state_interface name="velocity">
             <param name="initial_value">0.0</param>
+          </state_interface>
           <state_interface name="effort"/>
         </joint>
@@ -99,19 +134,21 @@
           <xacro:configure_joint joint_name="${name_stem}joint6" initial_position="${pi/2}"/>
           <xacro:configure_joint joint_name="${name_stem}joint7" initial_position="${pi/4}"/>
-          <xacro:if value="${gazebo and hand}">
+          <xacro:if value="${(gazebo or use_mujoco) and hand}">
             <xacro:configure_joint joint_name="${name_stem}finger_joint1" initial_position="0.0" />
           </xacro:if>
-          <!-- Cartesian velocity interfaces -->
-          <xacro:general_purpose_io prefix="${arm_prefix}vx" command_interface="cartesian_velocity" index="0"/>
-          <xacro:general_purpose_io prefix="${arm_prefix}vy" command_interface="cartesian_velocity" index="1"/>
-          <xacro:general_purpose_io prefix="${arm_prefix}vz" command_interface="cartesian_velocity" index="2"/>
-          <xacro:general_purpose_io prefix="${arm_prefix}wx" command_interface="cartesian_velocity" index="3"/>
-          <xacro:general_purpose_io prefix="${arm_prefix}wy" command_interface="cartesian_velocity" index="4"/>
-          <xacro:general_purpose_io prefix="${arm_prefix}wz" command_interface="cartesian_velocity" index="5"/>
-          <!-- Cartesian pose interfaces, in total 16 interfaces -->
-          <xacro:pose_loop name_stem="${arm_prefix}" i="0"/>
-          <!-- Elbow command interfaces -->
-          <xacro:general_purpose_io prefix="${arm_prefix}joint_3_position" command_interface="elbow_command" index="0"/>
-          <xacro:general_purpose_io prefix="${arm_prefix}joint_4_sign" command_interface="elbow_command" index="1"/>
+          <xacro:unless value="${use_mujoco}">
+            <!-- Cartesian velocity interfaces -->
+            <xacro:general_purpose_io prefix="${arm_prefix}vx" command_interface="cartesian_velocity" index="0"/>
+            <xacro:general_purpose_io prefix="${arm_prefix}vy" command_interface="cartesian_velocity" index="1"/>
+            <xacro:general_purpose_io prefix="${arm_prefix}vz" command_interface="cartesian_velocity" index="2"/>
+            <xacro:general_purpose_io prefix="${arm_prefix}wx" command_interface="cartesian_velocity" index="3"/>
+            <xacro:general_purpose_io prefix="${arm_prefix}wy" command_interface="cartesian_velocity" index="4"/>
+            <xacro:general_purpose_io prefix="${arm_prefix}wz" command_interface="cartesian_velocity" index="5"/>
+            <!-- Cartesian pose interfaces, in total 16 interfaces -->
+            <xacro:pose_loop name_stem="${arm_prefix}" i="0"/>
+            <!-- Elbow command interfaces -->
+            <xacro:general_purpose_io prefix="${arm_prefix}joint_3_position" command_interface="elbow_command" index="0"/>
+            <xacro:general_purpose_io prefix="${arm_prefix}joint_4_sign" command_interface="elbow_command" index="1"/>
+          </xacro:unless>
           <xacro:robot_loop i="${i+1}"/>
         </xacro:unless>

File: robots/common/franka_multi_robot.xacro (robot description, xacro)
@@ -23,4 +23,5 @@
                       with_sc:='false'
                       ros2_control:=false
+                      use_mujoco:=false
                       robot_ips:=''
                       use_fake_hardware:=false
@@ -181,4 +182,5 @@
           hand="${hand}"
           gazebo_effort="${gazebo_effort}"
+          use_mujoco="${use_mujoco}"
       />
     </xacro:if>

File: robots/common/franka_robot.xacro (robot description, xacro)
@@ -23,5 +23,4 @@
                       ros2_control:=false
                       use_mujoco:=false
-                      mujoco_scene_xacro_path:=''
                       robot_ip:=''
                       use_fake_hardware:=false
@@ -159,12 +158,4 @@
           use_mujoco="${use_mujoco}"
           no_prefix="${no_prefix}"
-          connected_to="${connected_to}"
-          xyz="${xyz}"
-          rpy="${rpy}"
-          ee_id="${ee_id}"
-          xyz_ee="${xyz_ee}"
-          rpy_ee="${rpy_ee}"
-          tcp_xyz="${tcp_xyz}"
-          tcp_rpy="${tcp_rpy}"
       />
     </xacro:if>

File: robots/fr3/fr3.urdf.xacro (robot description, xacro)
@@ -34,6 +34,4 @@
   <xacro:arg name="ros2_control" default="false" />
   <xacro:arg name="use_mujoco" default="false" />
-  <!-- MuJoCo scene XML string (generated from mujoco_scene_xacro in the launch file) -->
-  <xacro:arg name="mujoco_scene_xacro_path" default="" />
   <!-- IP address or hostname of the robot" -->
   <xacro:arg name="robot_ip" default="" />
@@ -69,5 +67,4 @@
                       ros2_control="$(arg ros2_control)"
                       use_mujoco="$(arg use_mujoco)"
-                      mujoco_scene_xacro_path="$(arg mujoco_scene_xacro_path)"
                       robot_ip="$(arg robot_ip)"
                       use_fake_hardware="$(arg use_fake_hardware)"
